Commit message: edit joint name

File: sentinel_description/urdf/sentinel.xacro (robot description, xacro)
@@ -17,5 +17,5 @@
         <origin xyz="0.0 0.0 0.04" rpy="0.0 0.0 0.0"/>
     </joint>
-    <joint name="top_right_wheel_joint" type="continuous">
+    <joint name="fr_motor_joint" type="continuous">
         <parent link="base_link"/>
         <child link="top_right_wheel"/>
@@ -23,5 +23,5 @@
         <origin xyz="0.105 -0.125 -0.01" rpy="-1.57079632679  0 0"/>
     </joint>
-    <joint name="top_left_wheel_joint" type="continuous">
+    <joint name="fl_motor_joint" type="continuous">
         <parent link="base_link"/>
         <child link="top_left_wheel"/>
@@ -29,5 +29,5 @@
         <origin xyz="0.105 0.125 -0.01" rpy="-1.57079632679  0 0"/>
     </joint>
-    <joint name="lower_right_wheel_joint" type="continuous">
+    <joint name="lr_motor_joint" type="continuous">
         <parent link="base_link"/>
         <child link="lower_right_wheel"/>
@@ -35,5 +35,5 @@
         <origin xyz="-0.105 -0.125 -0.01" rpy="-1.57079632679  0 0"/>
     </joint>
-    <joint name="lower_left_wheel_joint" type="continuous">
+    <joint name="ll_motor_joint" type="continuous">
         <parent link="base_link"/>
         <child link="lower_left_wheel"/>
